File: pico_debug/pico_debug.kicad_pcb (KiCad board)
At the start: 2 copper layers, 95 x 55 mm, 12 parts, among them SW3 SW_SPST

Commit message: PCB updates for v2
Parts:
- R1: footprint Resistor_THT:R_Axial_DIN0204_L3.6mm_D1.6mm_P7.62mm_Horizontal -> Resistor_THT:R_Axial_DIN0207_L6.3mm_D2.5mm_P10.16mm_Horizontal
- moved R1 4.52 mm to (135.0, 92.6)
Routing:
- net Net-(A1-GPIO12): track 36.6 -> 40.1 mm
Other:
- board text added: "Debug Probe"
- board text added: "Target"
- board text added: "pico_debug v2 yarg-lang.dev John McAleely 2026"
- board text removed: "pico_debug v1 yarg-lang.dev John McAleely 2026"
