File: pico_debug/pico_debug.kicad_sch (KiCad schematic)
At the start: 12 parts, among them J1 Conn_02x03_Counter_Clockwise, SW1 SW_SPST, SW2 SW_SPST, SW3 SW_SPST

Commit message: v1 sent to pcbway
Parts:
- H1, H2, H3, H4: footprint MountingHole:MountingHole_3.2mm_M3 -> MountingHole:MountingHole_3.2mm_M3_Pad_Via
Other:
- moved on the sheet: D1, J1, R1, SW1, SW2, SW3
